Commit message: sync https://www.lejuhub.com/highlydynamic/kuavo-ros-control/commit/cd177261414262200d77006d43afe5ad39e4e811

File: src/kuavo_assets/models/biped_s31/urdf/biped_s31.urdf (robot description, URDF)
Before this commit: robot biped_s31, 28 links, 27 joints
Joints:
- removed joint dummy_to_base_link
- added joint base_link_to_dummy_link: type fixed, parent base_link, child dummy_link, origin xyz=0 0 0 rpy=0 0 0

File: src/kuavo_assets/models/biped_s32/urdf/biped_s32.urdf (robot description, URDF)
Before this commit: robot biped_s32, 28 links, 27 joints
Joints:
- removed joint dummy_to_base_link
- added joint base_link_to_dummy_link: type fixed, parent base_link, child dummy_link, origin xyz=0 0 0 rpy=0 0 0

File: src/kuavo_assets/models/biped_s43/urdf/biped_s43.urdf (robot description, URDF)
Before this commit: robot biped_s43, 46 links, 45 joints
Joints:
- removed joint dummy_to_base_link
- added joint base_link_to_dummy_link: type fixed, parent base_link, child dummy_link, origin xyz=0 0 0 rpy=0 0 0

File: src/kuavo_assets/models/biped_s45/urdf/biped_s45.urdf (robot description, URDF)
Before this commit: robot biped_s45, 47 links, 46 joints
Links:
- added link torso-camera, mass 0.1; collision mesh filename=package://kuavo_assets/models/biped_s45/meshes/torso-camera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; visual mesh filename=package://kuavo_assets/models/biped_s45/meshes/torso-camera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
- added link waist_camera, mass 0.237986769607677; collision mesh filename=package://kuavo_assets/models/biped_s45/meshes/waist_camera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; visual mesh filename=package://kuavo_assets/models/biped_s45/meshes/waist_camera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
- link base_link: mass 22.11293803 -> 21.77493803
Joints:
- removed joint dummy_to_base_link
- added joint base_link_to_dummy_link: type fixed, parent base_link, child dummy_link, origin xyz=0 0 0 rpy=0 0 0
- added joint torso-camera: type fixed, parent base_link, child torso-camera, origin xyz=0.115535332475413 0.0175000000005085 0.2883441440894 rpy=0 0.732666 0, axis 0 0 0
- added joint waist_camera: type fixed, parent base_link, child waist_camera, origin xyz=0.168717483101422 0 0.01355599662743 rpy=0 0 0, axis 0 0 0

File: src/kuavo_assets/models/biped_s45/urdf/biped_s45_gazebo.urdf (robot description, URDF)
Before this commit: robot biped_s45, 47 links, 46 joints
Joints:
- joint l_foot_heel_joint: origin xyz=-0.073164 0.0 -0.0595 rpy=0 0 0 -> xyz=-0.0 0.04773 -0.0595 rpy=0 0 0
- joint l_foot_toe_joint: origin xyz=0.17084 0.0 -0.0595 rpy=0 0 0 -> xyz=0.0 -0.04773 -0.0595 rpy=0 0 0
- joint r_foot_heel_joint: origin xyz=-0.073164 0.0 -0.0595 rpy=0 0 0 -> xyz=-0.0 0.04773 -0.0595 rpy=0 0 0
- joint r_foot_toe_joint: origin xyz=0.17084 0.0 -0.0595 rpy=0 0 0 -> xyz=0.0 -0.04773 -0.0595 rpy=0 0 0

File: src/kuavo_assets/models/biped_s47/urdf/biped_s47.urdf (robot description, URDF)
Before this commit: robot biped_s47, 62 links, 61 joints
Joints:
- joint zarm_l7_end_effector_joint: origin xyz=0 -0.03 -0.17 rpy=0 0 0 -> xyz=0 -0.0 -0.17 rpy=0 0 0
- joint zarm_r7_end_effector_joint: origin xyz=0 0.03 -0.17 rpy=0 0 0 -> xyz=0 0.0 -0.17 rpy=0 0 0

File: src/kuavo_assets/models/biped_s48/urdf/biped_s48.urdf (robot description, URDF)
Before this commit: robot biped_s48, 69 links, 68 joints
Joints:
- removed joint dummy_to_base_link
- added joint base_link_to_dummy_link: type fixed, parent base_link, child dummy_link, origin xyz=0 0 0 rpy=0 0 0

File: src/kuavo_assets/models/biped_s49/urdf/biped_s49.urdf (robot description, URDF)
Before this commit: robot biped_s49, 47 links, 46 joints
Joints:
- removed joint dummy_to_base_link
- added joint base_link_to_dummy_link: type fixed, parent base_link, child dummy_link, origin xyz=0 0 0 rpy=0 0 0
