Commit message: sync https://www.lejuhub.com/highlydynamic/kuavo-ros-control/commit/5b8e8c229c12a4cf6c0f2d2935e5512670dcbace

File: src/gazebo/realsense_ros_gazebo/xacro/depthcam.xacro (robot description, xacro)
@@ -129,5 +129,5 @@
         <always_on>1</always_on>
         <update_rate>15</update_rate>
-        <visualize>1</visualize>
+        <visualize>0</visualize>
       </sensor>
       <sensor name="${sensor_name}_ired1" type="camera">
@@ -313,5 +313,5 @@
               <always_on>1</always_on>
               <update_rate>${rate}</update_rate>
-              <visualize>1</visualize>
+              <visualize>0</visualize>
           </sensor>
           <sensor name="${sensor_name}_ired1" type="camera">

File: src/kuavo_assets/models/biped_s40/urdf/biped_s40.urdf (robot description, URDF)
Before this commit: robot biped_s40, 46 links, 45 joints
Joints:
- removed joint dummy_to_base_link
- added joint base_link_to_dummy_link: type fixed, parent base_link, child dummy_link, origin xyz=0 0 0 rpy=0 0 0

File: src/kuavo_assets/models/biped_s41/urdf/biped_s41.urdf (robot description, URDF)
Before this commit: robot biped_s41, 46 links, 45 joints
Joints:
- removed joint dummy_to_base_link
- added joint base_link_to_dummy_link: type fixed, parent base_link, child dummy_link, origin xyz=0 0 0 rpy=0 0 0

File: src/kuavo_assets/models/biped_s42/urdf/biped_s42.urdf (robot description, URDF)
Before this commit: robot biped_s42, 47 links, 46 joints
Joints:
- removed joint dummy_to_base_link
- added joint base_link_to_dummy_link: type fixed, parent base_link, child dummy_link, origin xyz=0 0 0 rpy=0 0 0

File: src/kuavo_assets/models/biped_s43/urdf/biped_s43.urdf (robot description, URDF)
Before this commit: robot biped_s43, 46 links, 45 joints
Links:
- link base_link: geometry collision cylinder length=0.5 radius=0.15; visual mesh filename=package://kuavo_assets/models/biped_s43/meshes/base_link.STL
- link zarm_l2_link: geometry collision cylinder length=0.3 radius=0.05; visual mesh filename=package://kuavo_assets/models/biped_s43/meshes/l_arm_roll.S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
- link zarm_l4_link: geometry collision cylinder length=0.26 radius=0.05; visual mesh filename=package://kuavo_assets/models/biped_s43/meshes/l_forearm.STL
- link zarm_l7_link: geometry collision cylinder length=0.14 radius=0.04; visual mesh filename=package://kuavo_assets/models/biped_s43/meshes/l_hand_pitch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
- link zarm_r2_link: geometry collision cylinder length=0.3 radius=0.05; visual mesh filename=package://kuavo_assets/models/biped_s43/meshes/r_arm_roll.S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
- link zarm_r4_link: geometry collision cylinder length=0.26 radius=0.05; visual mesh filename=package://kuavo_assets/models/biped_s43/meshes/r_forearm.STL
- link zarm_r7_link: geometry collision cylinder length=0.14 radius=0.04; visual mesh filename=package://kuavo_assets/models/biped_s43/meshes/r_hand_pitch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
- link zhead_1_link: geometry collision sphere radius=0.1; visual mesh filename=package://kuavo_assets/models/biped_s43/meshes/head_yaw.STL
Joints:
- removed joint dummy_to_base_link
- added joint base_link_to_dummy_link: type fixed, parent base_link, child dummy_link, origin xyz=0 0 0 rpy=0 0 0

File: src/kuavo_assets/models/biped_s45/urdf/biped_s45.urdf (robot description, URDF)
Before this commit: robot biped_s45, 47 links, 46 joints
Links:
- added link l_hand_camera, mass 0.038145442577304; collision mesh filename=package://kuavo_assets/models/biped_s45/meshes/l_hand_camer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; visual mesh filename=package://kuavo_assets/models/biped_s45/meshes/l_hand_camer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
- added link l_hand_tripod, mass 0.0342669089979502; collision mesh filename=package://kuavo_assets/models/biped_s45/meshes/l_hand_tripo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; visual mesh filename=package://kuavo_assets/models/biped_s45/meshes/l_hand_tripo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
- added link r_hand_camera, mass 0.038145442577304; collision mesh filename=package://kuavo_assets/models/biped_s45/meshes/r_hand_camer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; visual mesh filename=package://kuavo_assets/models/biped_s45/meshes/r_hand_camer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
- added link r_hand_tripod, mass 0.034266881719861; collision mesh filename=package://kuavo_assets/models/biped_s45/meshes/r_hand_tripo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; visual mesh filename=package://kuavo_assets/models/biped_s45/meshes/r_hand_tripo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
- added link torso-camera, mass 0.1; collision mesh filename=package://kuavo_assets/models/biped_s45/meshes/torso-camera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; visual mesh filename=package://kuavo_assets/models/biped_s45/meshes/torso-camera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
- added link waist_camera, mass 0.237986769607677; collision mesh filename=package://kuavo_assets/models/biped_s45/meshes/waist_camera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; visual mesh filename=package://kuavo_assets/models/biped_s45/meshes/waist_camera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
- link base_link: mass 22.11293803 -> 27.41553803; geometry collision cylinder length=0.6 radius=0.15; visual mesh filename=package://kuavo_assets/models/biped_s45/meshes/torso.STL
- link zarm_l2_link: geometry collision cylinder length=0.3 radius=0.05; visual mesh filename=package://kuavo_assets/models/biped_s45/meshes/l_arm_roll.S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
- link zarm_l4_link: geometry collision cylinder length=0.26 radius=0.05; visual mesh filename=package://kuavo_assets/models/biped_s45/meshes/l_forearm.STL
- link zarm_l7_end_effector: geometry collision sphere radius=0.01
- link zarm_l7_link: geometry collision cylinder length=0.14 radius=0.04; visual mesh filename=package://kuavo_assets/models/biped_s45/meshes/l_hand_pitch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
- link zarm_r2_link: geometry collision cylinder length=0.3 radius=0.05; visual mesh filename=package://kuavo_assets/models/biped_s45/meshes/r_arm_roll.S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
- link zarm_r4_link: geometry collision cylinder length=0.26 radius=0.05; visual mesh filename=package://kuavo_assets/models/biped_s45/meshes/r_forearm.STL
- link zarm_r7_end_effector: geometry collision sphere radius=0.01
- link zarm_r7_link: geometry collision cylinder length=0.14 radius=0.04; visual mesh filename=package://kuavo_assets/models/biped_s45/meshes/r_hand_pitch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
- link zhead_1_link: geometry collision sphere radius=0.1; visual mesh filename=package://kuavo_assets/models/biped_s45/meshes/head_yaw.STL
Joints:
- removed joint dummy_to_base_link
- added joint base_link_to_dummy_link: type fixed, parent base_link, child dummy_link, origin xyz=0 0 0 rpy=0 0 0
- added joint l_hand_camera_joint: type fixed, parent l_hand_tripod, child l_hand_camera, origin xyz=0.11540559159102 -0.0145586110669961 -0.110123491595499 rpy=1.919862177193763 0.753528063917894 -2.897246568680842, axis 0 0 0
- added joint l_hand_tripod_joint: type fixed, parent zarm_l7_link, child l_hand_tripod, origin xyz=0.0 0.0 0.0 rpy=0.0 0.0 0.0, axis 0 0 0
- added joint r_hand_camera_joint: type fixed, parent r_hand_tripod, child r_hand_camera, origin xyz=0.115405591590931 0.0154312352120435 -0.107724128430896 rpy=1.208853693239594  0.751879414295006 2.888346587751982, axis 0 0 0
- added joint r_hand_tripod_joint: type fixed, parent zarm_r7_link, child r_hand_tripod, origin xyz=0.0 0.0 0.0 rpy=0.0 0.0 0.0, axis 0 0 0
- added joint torso-camera: type fixed, parent base_link, child torso-camera, origin xyz=0.115535332475413 0.0175000000005085 0.2883441440894 rpy=0 0.732666 0, axis 0 0 0
- added joint waist_camera: type fixed, parent base_link, child waist_camera, origin xyz=0.168717483101422 0 0.01355599662743 rpy=0 0 0, axis 0 0 0

File: src/kuavo_assets/models/biped_s45/urdf/biped_s45_gazebo.urdf (robot description, URDF)
Before this commit: robot biped_s45, 47 links, 46 joints
Links:
- link base_link: mass 22.11293803 -> 27.89833803
Joints:
- joint l_foot_heel_joint: origin xyz=-0.073164 0.0 -0.0595 rpy=0 0 0 -> xyz=-0.0 0.04773 -0.0595 rpy=0 0 0
- joint l_foot_toe_joint: origin xyz=0.17084 0.0 -0.0595 rpy=0 0 0 -> xyz=0.0 -0.04773 -0.0595 rpy=0 0 0
- joint r_foot_heel_joint: origin xyz=-0.073164 0.0 -0.0595 rpy=0 0 0 -> xyz=-0.0 0.04773 -0.0595 rpy=0 0 0
- joint r_foot_toe_joint: origin xyz=0.17084 0.0 -0.0595 rpy=0 0 0 -> xyz=0.0 -0.04773 -0.0595 rpy=0 0 0

File: src/kuavo_assets/models/biped_s45/urdf/drake/biped_v3.urdf (robot description, URDF)
Before this commit: robot biped_v3, 13 links, 12 joints
Links:
- link torso: mass 33.72893803 -> 39.51433803

File: src/kuavo_assets/models/biped_s45/urdf/drake/biped_v3_all_joint.urdf (robot description, URDF)
Before this commit: robot biped_v3_all_joint, 35 links, 30 joints
Links:
- link torso: mass 22.70214316 -> 28.48754316

File: src/kuavo_assets/models/biped_s45/urdf/drake/biped_v3_full.urdf (robot description, URDF)
Before this commit: robot biped_v3_full, 27 links, 26 joints
Links:
- link torso: mass 23.34493803 -> 29.13033803

File: src/kuavo_assets/models/biped_s46/urdf/biped_s46.urdf (robot description, URDF)
Before this commit: robot biped_s46, 46 links, 45 joints
Links:
- link base_link: geometry collision cylinder length=0.6 radius=0.15; visual mesh filename=package://kuavo_assets/models/biped_s46/meshes/torso.STL
- link zarm_l2_link: geometry collision cylinder length=0.3 radius=0.05; visual mesh filename=package://kuavo_assets/models/biped_s46/meshes/l_arm_roll.S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
- link zarm_l4_link: geometry collision cylinder length=0.26 radius=0.05; visual mesh filename=package://kuavo_assets/models/biped_s46/meshes/l_forearm.STL
- link zarm_l7_link: geometry collision cylinder length=0.14 radius=0.04; visual mesh filename=package://kuavo_assets/models/biped_s46/meshes/l_hand_pitch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
- link zarm_r2_link: geometry collision cylinder length=0.3 radius=0.05; visual mesh filename=package://kuavo_assets/models/biped_s46/meshes/r_arm_roll.S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
- link zarm_r4_link: geometry collision cylinder length=0.26 radius=0.05; visual mesh filename=package://kuavo_assets/models/biped_s46/meshes/r_forearm.STL
- link zarm_r7_link: geometry collision cylinder length=0.14 radius=0.04; visual mesh filename=package://kuavo_assets/models/biped_s46/meshes/r_hand_pitch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
- link zhead_1_link: geometry collision sphere radius=0.12; visual mesh filename=package://kuavo_assets/models/biped_s46/meshes/head_yaw.STL

File: src/kuavo_assets/models/biped_s47/urdf/biped_s47.urdf (robot description, URDF)
Before this commit: robot biped_s47, 62 links, 61 joints
Links:
- link base_link: geometry collision cylinder length=0.6 radius=0.15; visual mesh filename=package://kuavo_assets/models/biped_s47/meshes/torso.STL
- link zarm_l2_link: geometry collision cylinder length=0.3 radius=0.05; visual mesh filename=package://kuavo_assets/models/biped_s47/meshes/l_arm_roll.S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
- link zarm_l4_link: geometry collision cylinder length=0.26 radius=0.05; visual mesh filename=package://kuavo_assets/models/biped_s47/meshes/l_forearm.STL
- link zarm_l7_link: geometry collision cylinder length=0.14 radius=0.04; visual mesh filename=package://kuavo_assets/models/biped_s47/meshes/l_hand_pitch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
- link zarm_r2_link: geometry collision cylinder length=0.3 radius=0.05; visual mesh filename=package://kuavo_assets/models/biped_s47/meshes/r_arm_roll.S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
- link zarm_r4_link: geometry collision cylinder length=0.26 radius=0.05; visual mesh filename=package://kuavo_assets/models/biped_s47/meshes/r_forearm.STL
- link zarm_r7_link: geometry collision cylinder length=0.14 radius=0.04; visual mesh filename=package://kuavo_assets/models/biped_s47/meshes/r_hand_pitch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
- link zhead_1_link: geometry collision sphere radius=0.1; visual mesh filename=package://kuavo_assets/models/biped_s47/meshes/head_yaw.STL
Joints:
- joint zarm_l7_end_effector_joint: origin xyz=0 -0.03 -0.17 rpy=0 0 0 -> xyz=0 -0.0 -0.17 rpy=0 0 0
- joint zarm_r7_end_effector_joint: origin xyz=0 0.03 -0.17 rpy=0 0 0 -> xyz=0 0.0 -0.17 rpy=0 0 0

File: src/kuavo_assets/models/biped_s48/urdf/biped_s48.urdf (robot description, URDF)
Before this commit: robot biped_s48, 69 links, 68 joints
Links:
- link base_link: mass 22.11293803 -> 27.41553803; geometry collision cylinder length=0.6 radius=0.15; visual mesh filename=package://kuavo_assets/models/biped_s48/meshes/torso.STL
- link zarm_l2_link: geometry collision cylinder length=0.3 radius=0.05; visual mesh filename=package://kuavo_assets/models/biped_s48/meshes/l_arm_roll.S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
- link zarm_l4_link: geometry collision cylinder length=0.26 radius=0.05; visual mesh filename=package://kuavo_assets/models/biped_s48/meshes/l_forearm.STL
- link zarm_l7_link: geometry collision cylinder length=0.14 radius=0.04; visual mesh filename=package://kuavo_assets/models/biped_s48/meshes/l_hand_pitch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
- link zarm_r2_link: geometry collision cylinder length=0.3 radius=0.05; visual mesh filename=package://kuavo_assets/models/biped_s48/meshes/r_arm_roll.S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
- link zarm_r4_link: geometry collision cylinder length=0.26 radius=0.05; visual mesh filename=package://kuavo_assets/models/biped_s48/meshes/r_forearm.STL
- link zarm_r7_link: geometry collision cylinder length=0.14 radius=0.04; visual mesh filename=package://kuavo_assets/models/biped_s48/meshes/r_hand_pitch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
- link zhead_2_link: geometry collision sphere radius=0.1; visual mesh filename=package://kuavo_assets/models/biped_s48/meshes/head_pitch.S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
Joints:
- removed joint dummy_to_base_link
- added joint base_link_to_dummy_link: type fixed, parent base_link, child dummy_link, origin xyz=0 0 0 rpy=0 0 0
