Commit message: sync https://www.lejuhub.com/highlydynamic/kuavo-ros-control/commit/f2b748d5e6402da55b8bd21a9d3de95f8d3506a2

File: src/kuavo_assets/models/apriltag/urdf/apriltag.xacro (robot description, xacro)
@@ -1,5 +1,5 @@
 <?xml version="1.0"?>
 <robot xmlns:xacro="http://ros.org/wiki/xacro" name="apriltag_marker">
-  <xacro:macro name="apriltag_marker" params="parent_link *origin id">
+  <xacro:macro name="apriltag_marker" params="parent_link *origin id enable_collision:=true">
     <!-- 定义二维码的Link -->
     <link name="apriltag_marker_${id}">
@@ -10,9 +10,11 @@
         </geometry>
       </visual>
-      <collision>
-        <geometry>
-          <box size="0.11 0.11 0.001"/>
-        </geometry>
-      </collision>
+      <xacro:if value="${enable_collision}">
+        <collision>
+          <geometry>
+            <box size="0.11 0.11 0.001"/>
+          </geometry>
+        </collision>
+      </xacro:if>
     </link>
     <joint name="apriltag_joint_${id}" type="fixed">
