Commit message: sync https://www.lejuhub.com/highlydynamic/kuavo-ros-control/commit/cb2f632a531bd2c9c75333f70e86230773a5f231

File: src/kuavo_assets/models/apriltag/urdf/block.urdf.xacro (robot description, xacro)
@@ -49,6 +49,8 @@
     <!-- 质量惯性（合并计算） -->
     <inertial>
-      <mass value="0.5"/>
-      <inertia ixx="0.0025" ixy="0" ixz="0" iyy="0.0025" iyz="0" izz="0.0025"/>
+      <!-- <mass value="0.5"/>
+      <inertia ixx="0.0025" ixy="0" ixz="0" iyy="0.0025" iyz="0" izz="0.0025"/> -->
+      <mass value="0.01"/>
+      <inertia ixx="0.00001" ixy="0" ixz="0" iyy="0.00001" iyz="0" izz="0.00001"/>
     </inertial>
   </link>
@@ -59,3 +61,14 @@
     <origin xyz="0 -1.0 0.9" rpy="0 0 0"/>
   </joint>
+  <!-- Gazebo物理属性配置 -->
+  <gazebo reference="base_link">
+    <material>Gazebo/Red</material>
+    <mu1>0.8</mu1>
+    <mu2>0.8</mu2>
+    <kp>1000000.0</kp>
+    <kd>100.0</kd>
+    <minDepth>0.001</minDepth>
+    <maxVel>1.0</maxVel>
+    <maxContacts>20</maxContacts>
+  </gazebo>
 </robot>

File: src/kuavo_assets/models/biped_s45/urdf/biped_s45_gazebo.urdf (robot description, URDF)
Before this commit: robot biped_s45, 47 links, 46 joints
Links:
- link base_link: mass 27.89833803 -> 22.11293803
- link zarm_l7_link: geometry collision mesh filename=package://kuavo_assets/models/biped_s45/meshes/l_hand_pitch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; visual mesh filename=package://kuavo_assets/models/biped_s45/meshes/l_hand_pitch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
- link zarm_r7_link: geometry collision mesh filename=package://kuavo_assets/models/biped_s45/meshes/r_hand_pitch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; visual mesh filename=package://kuavo_assets/models/biped_s45/meshes/r_hand_pitch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
