Commit message: sync https://www.lejuhub.com/highlydynamic/kuavo-ros-control/commit/fa211817a463596a6e35ea65d7aaea21b31350d6

File: src/kuavo_assets/models/biped_s13/urdf/biped_s13.urdf (robot description, URDF)
Before this commit: robot biped_s13, 39 links, 38 joints
Links:
- link leg_l6_link: geometry collision box size=0.21 0.1 0.035; visual mesh filename=package://kuavo_assets/models/biped_s13/meshes/l_foot_roll_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
- link leg_r6_link: geometry collision box size=0.21 0.1 0.035; visual mesh filename=package://kuavo_assets/models/biped_s13/meshes/r_foot_roll_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

File: src/kuavo_assets/models/biped_s14/urdf/biped_s14.urdf (robot description, URDF)
Before this commit: robot biped_s14, 39 links, 38 joints
Links:
- link leg_l6_link: geometry collision box size=0.205 0.1 0.035; visual mesh filename=package://kuavo_assets/models/biped_s14/meshes/l_foot_roll.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
- link leg_r6_link: geometry collision box size=0.205 0.1 0.035; visual mesh filename=package://kuavo_assets/models/biped_s14/meshes/r_foot_roll.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
